File: mark-4/CowPi-mk4b/CowPi-mk4b.kicad_sch (KiCad schematic)
At the start: 76 parts, among them J1 Conn_01x04_Pin, U1 TS-1187A-B-A-B, U10 1N4001_C2892326, U11 TS-1187A-B-A-B, U12 1N4001_C2892326, U13 TS-1187A-B-A-B, U14 1N4001_C2892326, U15 TS-1187A-B-A-B, U16 1N4001_C2892326, U17 TS-1187A-B-A-B, U18 TS-1187A-B-A-B, U19 1N4001_C2892326, U2 1N4001_C2892326, U20 1N4001_C2892326, U21 TS-1187A-B-A-B, U22 TS-1187A-B-A-B, U23 1N4001_C2892326, U24 1N4001_C2892326, U25 TS-1187A-B-A-B, U26 TS-1187A-B-A-B, U27 1N4001_C2892326, U28 1N4001_C2892326, U29 TS-1187A-B-A-B, U3 TS-1187A-B-A-B, U30 TS-1187A-B-A-B, U31 1N4001_C2892326, U32 1N4001_C2892326, U33 TS-1187A-B-A-B, U34 TS-1187A-B-A-B, U35 SS-3390S-L0, U36 SS-3390S-L0, U37 TS-1187A-B-A-B, U38 X6511FRS-11-C85D30, U39 X6511FRS-11-C85D30, U4 1N4001_C2892326, U40 BSS138_C3015220, U41 BSS138_C3015220, U42 BSS138_C3015220, U43 BSS138_C3015220, U44 HS96L03W2C03, U45 Pico, U46 BSS138_C3015220, U47 BSS138_C3015220, U48 BSS138_C3015220, U5 TS-1187A-B-A-B, U6 1N4001_C2892326, U7 TS-1187A-B-A-B, U8 1N4001_C2892326, U9 TS-1187A-B-A-B

Commit message: created version of mk3b that has through-holes for display module
Parts:
- J1: value Conn_01x04_Pin -> X6511WVS-04H-C60D48R2; footprint Connector_PinHeader_2.54mm:PinHeader_1x04_P2.54mm_Vertical_SMD_Pin1Right -> footprint:HDR-SMD_4P-P2.54-V-M-LS4.8_R2; symbol Connector:Conn_01x04_Pin -> X6511WVS-04H-C60D48R2:X6511WVS-04H-C60D48R2; LCSC (none) -> C2883761
Changed lines of the file:
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@@
     )
   )
-  (symbol (lib_id "Connector:Conn_01x04_Pin") (at 28.956 177.546 0) (unit 1)
-    (in_bom yes) (on_board yes) (dnp no) (fields_autoplaced)
-    (property "Reference" "J1" (at 29.591 170.942 0)
-      (effects (font (size 1.27 1.27)))
+  (symbol (lib_id "X6511WVS-04H-C60D48R2:X6511WVS-04H-C60D48R2") (at 28.956 178.816 0) (mirror y) (unit 1)
+    (in_bom yes) (on_board yes) (dnp no)
+    (property "Reference" "J1" (at 29.718 186.69 0)
+      (effects (font (size 1.27 1.27)) (justify left))
     )
-    (property "Value" "Conn_01x04_Pin" (at 29.591 173.482 0)
-      (effects (font (size 1.27 1.27)))
+    (property "Value" "X6511WVS-04H-C60D48R2" (at 40.64 169.926 0)
+      (effects (font (size 1.27 1.27)) (justify left))
     )
-    (property "Footprint" "Connector_PinHeader_2.54mm:PinHeader_1x04_P2.54mm_Vertical_SMD_Pin1Right" (at 28.956 177.546 0)
+    (property "Footprint" "footprint:HDR-SMD_4P-P2.54-V-M-LS4.8_R2" (at 28.956 188.976 0)
+      (effects (font (size 1.27 1.27) italic) hide)
+    )
+    (property "Datasheet" "https://atta.szlcsc.com/upload/public/pdf/source/20200909/C780060_F941EB1B69F43B5D6329EAF74E2E27BB.pdf" (at 31.242 178.689 0)
+      (effects (font (size 1.27 1.27)) (justify left) hide)
+    )
+    (property "LCSC" "C2883761" (at 28.956 178.816 0)
       (effects (font (size 1.27 1.27)) hide)
     )
-    (property "Datasheet" "~" (at 28.956 177.546 0)
-      (effects (font (size 1.27 1.27)) hide)
-    )
