File: mark-4/CowPi-mk4b-natural/CowPi-mk4b-natural.kicad_pcb (KiCad board)
At the start: 2 copper layers, 185.4 x 75.9 mm, 79 parts, among them J1 PH-00015, U1 TS-1187A-B-A-B, U10 1N4001_C2892326, U11 TS-1187A-B-A-B, U12 1N4001_C2892326, U13 TS-1187A-B-A-B, U14 1N4001_C2892326, U15 TS-1187A-B-A-B, U16 1N4001_C2892326, U17 TS-1187A-B-A-B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

Commit message: Updated mk4b-natural with OSHW certification mark and with alternate slide-switches
Parts:
- added G***: LOGO, art:OSHW-mk4b, B.Cu at (171.0, 81.5)
